File: hardware/review/ch32-pico.kicad_pcb (KiCad board)
At the start: 4 copper layers, 21 x 51 mm, 52 parts, among them J1 PICO 40-PIN, J2 GT-USB-7010AW, SW1 RESET, SW2 BOOT, U1 CH32X035C8T6, U4 AP63203WU-7

Commit message: Move SJ1 to the front, switch to the Basic tactile switch and refresh stock
The PC7 solder jumper now sits on the front beside the right header row
below the MCU, where it can be bridged without flipping the board; the
silkscreen audit and docs follow it. The board is rerouted with the pinned
Freerouting run, re-stitched and re-reviewed with DRC and connectivity clean.

RESET and BOOT use XUNPU TS-1088-AR02016 (C720477), a JLC Basic part with
the same land pattern as the 2.5 mm variant that showed no stock at order
time. The JLC procurement snapshot is refreshed: every fitted part now shows
stock for the batch, including the CH32X035 that was previously short, and
the parts estimate is $3.17 per board at 20.
Parts:
- SJ1: moved to F.Cu
- moved SJ1 14.0 mm to (16.8, 35.0)
Routing:
- net PB12: track 20.2 -> 32.1 mm, vias 5 -> 3
- net GPIO35: track 13.7 -> 22.3 mm
- net PB5: track 25.2 -> 33.3 mm, vias 3 -> 5
- net PA1: track 22.4 -> 14.8 mm
- net BOOT_PULLUP: track 41.2 -> 35.5 mm, vias 2 -> 4
- net PA21: track 37.3 -> 42.7 mm, vias 2 -> 3
- net PB10: track 28.8 -> 32.9 mm, vias 1 -> 4
- net PA20: track 21.4 -> 25.2 mm
- net CC1: track 32.1 -> 35.8 mm
- net PA23: track 13.6 -> 10.6 mm, vias 1 -> 2
- net PC6: track 4.98 -> 7.88 mm
- net GND: track 48.6 -> 45.8 mm, vias 27 -> 26
- net PA19: track 13.3 -> 15.9 mm
- net PA18: track 11.5 -> 14.2 mm
- net PA3: track 11.2 -> 13.8 mm
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
Commit message: Replace the AP63203 with a Silergy SY8301 buck
U4 is now the SY8301ABC: 4.5-40 V input, 1 A, 2 MHz, 22 uA quiescent, at
$0.18 instead of $1.06 at this quantity. R13/R14 (47k/15k) set 3.31 V from
its 0.8 V reference, with the top resistor sensing the output capacitors over
a dedicated bottom-layer trace that the shared pour must not bypass. R15
pulls EN up to the diode-OR node so VSYS-only power still starts the
regulator while header pin 37 grounds it. The inductor, bootstrap and bulk
capacitors are unchanged.

The SOT-23-6 pin order differs from the AP63203, so the cluster is re-laid
out: bootstrap capacitor above the IC, input capacitor below with ground
vias beside both it and the IC ground pin, inductor to the right, feedback
resistors on the left away from the switch node, enable pull-up and D4
below. The VBUS sense divider moves beside the connector and its probe pad
to the connector's left. The board is rerouted with the pinned Freerouting
run plus one KRT pass for the BOOT pull-up wire, re-stitched and re-reviewed
with DRC and connectivity clean; the power-layout audit now checks the
input-capacitor path and ground vias for this pinout. Library, render
model, procurement snapshot, cost figures and docs follow: parts are
$2.36 per board at 20.
Parts:
- added R13: 47k, ch32-pico:R0402, F.Cu at (3.60, 18.4)
- added R14: 15k, ch32-pico:R0402, F.Cu at (3.60, 16.8)
- added R15: 100k, ch32-pico:R0402, F.Cu at (10.2, 19.4)
- U4: value AP63203WU-7 -> SY8301ABC; footprint ch32-pico:TSOT-26_L2.9-W1.6-P0.95-LS2.8-BL -> ch32-pico:SOT-23-6_L2.9-W1.6-P0.95-LS2.8-BL
- moved C9 18.7 mm to (17.1, 7.40), turned to -90 degrees
- moved TP17 17.1 mm to (6.60, 4.60)
- moved R1 16.7 mm to (16.3, 6.20), turned to -90 degrees
- moved R2 16.6 mm to (16.3, 8.00), turned to -90 degrees
- moved D4 1.41 mm to (11.0, 21.0)
- moved C4 1.02 mm to (6.80, 12.9)
- moved C1 0.95 mm to (6.80, 18.6), turned to 180 degrees
- moved D1 0.81 mm to (3.50, 12.8)
Connections:
- U4 pad 1: 3V3_OUT -> BUCK_BST
- U4 pad 2: 3V3_EN -> GND
- U4 pad 3: VIN_SYS -> BUCK_FB
- U4 pad 4: GND -> 3V3_EN
- U4 pad 5: BUCK_SW -> VIN_SYS
- U4 pad 6: BUCK_BST -> BUCK_SW
Routing:
- net VBUS_SENSE: track 21.3 -> 41.1 mm
- net 3V3_OUT: track 76.4 -> 89.0 mm
- net GND: track 45.8 -> 55.0 mm, vias 26 -> 27
- net PA1: track 14.8 -> 23.5 mm, vias 2 -> 3
- net VBUS: track 60.7 -> 53.2 mm, vias 9 -> 8
- net VIN_SYS: track 9.59 -> 16.8 mm, vias 0 -> 2
- net GPIO35: track 22.3 -> 29.4 mm, vias 0 -> 1
- net PA11: track 17.8 -> 24.5 mm, vias 1 -> 4
- net PA20: track 25.2 -> 18.7 mm
- net PB5: track 33.3 -> 26.9 mm, vias 5 -> 3
- net PB13: track 26.8 -> 20.5 mm
- net PA2: track 18.3 -> 24.4 mm
- net PB8: track 22.6 -> 28.4 mm
- net 3V3_EN: track 17.4 -> 23.2 mm, vias 1 -> 3
- net CC1: track 35.8 -> 31.6 mm, vias 4 -> 3
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